Commit message: Update Genesis scene generation and SimFoundry asset workflows

File: self_improving/asset_pipeline/active/shared/openxsim/tests/fixtures/env_gen/fixture_assets/cabinet.urdf (robot description, URDF)
Before this commit: robot cabinet_fixture, 2 links, 1 joints
Links:
- removed link door
- added link drawer_1; visual box size=0.75 0.40 0.08
- added link drawer_2; visual box size=0.75 0.40 0.08
- added link drawer_3; visual box size=0.75 0.40 0.08
- link base: geometry visual box size=0.899 1.614 0.854
Joints:
- removed joint door_hinge
- added joint joint_1: type prismatic, parent base, child drawer_1, origin xyz=0 0.30 0, axis 0 0 -1, limit lower=0 upper=0.25 effort=100 velocity=1
- added joint joint_2: type prismatic, parent base, child drawer_2, origin xyz=0 0.807 0, axis 0 0 -1, limit lower=0 upper=0.25 effort=100 velocity=1
- added joint joint_3: type prismatic, parent base, child drawer_3, origin xyz=0 1.314 0, axis 0 0 -1, limit lower=0 upper=0.25 effort=100 velocity=1
